File: pure.kicad_pcb (KiCad board)
At the start: 2 copper layers, 100 x 90 mm, 146 parts, among them CON1 AVR-ISP-6, J1 JACK_TRS_3pins, J10 Conn_01x01, J11 Conn_01x01, J12 Conn_01x01, J13 Conn_Coaxial, J5 JACK_TRS_3pins, J7 ANT, J8 Jack-DC, J9 Conn_01x01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

Commit message: progress on schema
Parts:
- removed K2: RS-12, Relays_THT:Relay_DPDT_FRT5
- added C42: 47nF, LCSDR:C_1206_0603, F.Cu at (115.0, 140.1)
- added C44: 47pF, LCSDR:C_Disc_D7.5mm_W2.5mm_P5.00mm, F.Cu at (115.0, 140.1)
- added L12: 1uH, Inductors_THT:L_Axial_L12.8mm_D5.8mm_P20.32mm_Horizontal_Fastron_HBCC, F.Cu at (115.0, 140.1)
- added L2: 100uH, Inductors_THT:L_Axial_L5.3mm_D2.2mm_P7.62mm_Horizontal_Vishay_IM-1, F.Cu at (115.0, 140.1)
- added Q5: MMBT2222, LCSDR:SOT-23, F.Cu at (115.0, 140.1)
- added R40: 2.2k, LCSDR:R_1206_0603, F.Cu at (115.0, 140.1)
- added R41: 1k, LCSDR:R_0603_HandSoldering, F.Cu at (115.0, 140.1)
- added R42: 470, LCSDR:R_1206_0603, F.Cu at (115.0, 140.1)
- C15, C36, C73: footprint LCSDR:C_1206_0603 -> Capacitors_SMD:C_0603_HandSoldering
- C31: footprint LCSDR:C_0603_HandSoldering -> Capacitors_SMD:C_0603_HandSoldering
- K1: value TQ2-12VDC -> TIANBO-HJR-4102-L; footprint Relays_THT:Relay_DPDT_FRT5 -> Relays_THT:Relay_SPDT_HJR-4102
Connections:
- C15 pad 1: PA -> (no net)
- C39 pad 2: Net-(C39-Pad2) -> Relay
- C48 pad 2: Net-(C48-Pad2) -> IO_A
- C49 pad 2: Net-(C48-Pad2) -> IO_A
- D1 pad 2: Net-(C39-Pad2) -> Relay
- K1 pad 1: +12V -> (no net)
- K1 pad 5: (no net) -> +12V
- K1 pad 8: PA -> Relay
- Q3 pad 3: Net-(C39-Pad2) -> Relay
- Q4 pad 3: Net-(C37-Pad2) -> Net-(L12-Pad2)
- R10 pad 1: +12V -> (no net)
- R16 pad 1: Net-(C37-Pad2) -> Net-(L12-Pad2)
- R21 pad 1: Net-(C37-Pad2) -> Net-(L12-Pad2)
Routing:
- net RX90: track 0.00 -> 35.9 mm, vias 0 -> 2
- net Net-(Q2-Pad2): track 30.5 -> 0.00 mm
- net SCL: track 38.2 -> 11.9 mm
- net Net-(C32-Pad1): track 25.8 -> 0.00 mm
- net Net-(Q1-Pad2): track 38.7 -> 16.2 mm
- net +5V: track 24.4 -> 1.89 mm
- net SDA: track 31.0 -> 9.73 mm
- net PA: track 18.9 -> 0.00 mm
- net +12V: track 122.3 -> 136.6 mm
- net (no net): track 1038.4 -> 1051.5 mm, vias 59 -> 57
- net Net-(R26-Pad2): track 40.5 -> 28.7 mm
- net Net-(R1-Pad2): track 18.7 -> 9.13 mm
- net Net-(R28-Pad2): track 37.1 -> 28.2 mm
- net +3V3: track 97.2 -> 89.3 mm
- net TX_Q: track 8.12 -> 1.26 mm
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