File: pure.kicad_pcb (KiCad board)
At the start: 2 copper layers, 100 x 90 mm, 74 parts, among them J1 LINE_IN, J2 USB_B, J3 Program_USB_JTAG, K1 RS-12, Q1 DTC143Z, Q2 DTC143Z, Q3 BSS138, Q4 BSS138, Q5 DTC143Z, U1 SN74LVC1G3157DBVR, U11 CH340C, U2 SN74LVC1G3157DBVR, U3 74HC4053, U4 74HC4053, U5 MC33079, U6 ESP32-S3-WROOM-1-N16R8, U8 Si5351A-B-GT, U9 M24C01-WMN

Commit message: add custom footprints, progress on schema and PCB
Parts:
- added C26: 22..47nF, SDR_footprints:C_1206_0603, F.Cu at (164.6, 18.6)
- added C27: 390, SDR_footprints:C_1206_0603, F.Cu at (23.2, 155.2)
- added C28: 180, SDR_footprints:C_1206_0603, F.Cu at (23.2, 157.7)
- added C29: 390, SDR_footprints:C_1206_0603, F.Cu at (23.2, 160.2)
- added C30: 22..47nF, SDR_footprints:C_1206_0603, F.Cu at (10.4, 144.4)
- added C31: 100nF, SDR_footprints:C_1206_0603, F.Cu at (10.4, 147.0)
- added C32: 100nF, SDR_footprints:C_1206_0603, F.Cu at (164.2, 114.0)
- added C33: 360, Capacitor_SMD:C_0603_1608Metric_Pad1.08x0.95mm_HandSolder, F.Cu at (3.55, 155.2)
- added C34: 390, SDR_footprints:C_1206_0603, F.Cu at (3.55, 157.7)
- added C35: 100nF, SDR_footprints:C_1206_0603, F.Cu at (-23.4, 138.8)
- added C36: 360, SDR_footprints:C_1206_0603, F.Cu at (3.55, 160.2)
- added C37: 22..47nF, SDR_footprints:C_1206_0603, F.Cu at (-23.4, 141.3)
- added C39: 470, Capacitor_SMD:C_0603_1608Metric_Pad1.08x0.95mm_HandSolder, F.Cu at (35.6, 33.8)
- added C40: 470, SDR_footprints:C_1206_0603, F.Cu at (35.6, 36.3)
- added C41: 1nF, Capacitor_SMD:C_0603_1608Metric_Pad1.08x0.95mm_HandSolder, F.Cu at (15.9, 17.4)
- added C42: 560, Capacitor_SMD:C_0603_1608Metric_Pad1.08x0.95mm_HandSolder, F.Cu at (15.9, 19.9)
- added C43: 120, Capacitor_SMD:C_0603_1608Metric_Pad1.08x0.95mm_HandSolder, F.Cu at (15.9, 22.4)
- added C45: 1nF, Capacitor_SMD:C_0603_1608Metric_Pad1.08x0.95mm_HandSolder, F.Cu at (15.9, 24.9)
- added C46: 560, Capacitor_SMD:C_0603_1608Metric_Pad1.08x0.95mm_HandSolder, F.Cu at (15.9, 27.4)
- added C48: 560, Capacitor_SMD:C_0603_1608Metric_Pad1.08x0.95mm_HandSolder, F.Cu at (15.9, 29.9)
- added C49: 100nF, SDR_footprints:C_1206_0603, F.Cu at (44.6, 24.1)
- added C50: 100nF, SDR_footprints:C_1206_0603, F.Cu at (44.6, 26.6)
- added C51: 100nF, SDR_footprints:C_1206_0603, F.Cu at (44.6, 29.2)
- added D4: BAP50-03, Diode_SMD:D_SOD-323_HandSoldering, F.Cu at (10.3, 168.2)
- added D5: BAP50-03, Diode_SMD:D_SOD-323_HandSoldering, F.Cu at (10.3, 171.1)
- added D6: BAP50-03, Diode_SMD:D_SOD-323_HandSoldering, F.Cu at (-9.36, 168.2)
- added D7: BAP50-03, Diode_SMD:D_SOD-323_HandSoldering, F.Cu at (-9.36, 171.1)
- added D8: BAP50-03, Diode_SMD:D_SOD-323_HandSoldering, F.Cu at (20.7, 30.3)
- added D9: BAP50-03, Diode_SMD:D_SOD-323_HandSoldering, F.Cu at (20.7, 33.3)
- added L10: 0,47uH, SDR_footprints:Resistor_SMD+THTuniversal_0603to2512_RM10_HandSoldering, F.Cu at (9.30, 164.6)
- added L11: 1uH, SDR_footprints:Resistor_SMD+THTuniversal_0603to2512_RM10_HandSoldering, F.Cu at (-11.8, 150.5)
- added L12: 2,2uH, SDR_footprints:Resistor_SMD+THTuniversal_0603to2512_RM10_HandSoldering, F.Cu at (-10.4, 160.3)
- added L13: 1uH, SDR_footprints:Resistor_SMD+THTuniversal_0603to2512_RM10_HandSoldering, F.Cu at (-10.4, 164.6)
- added L14: 2,2uH, Inductor_THT:L_Axial_L6.6mm_D2.7mm_P10.16mm_Horizontal_Vishay_IM-2, F.Cu at (19.7, 18.2)
- added L15: 4,7uH, Inductor_THT:L_Axial_L6.6mm_D2.7mm_P10.16mm_Horizontal_Vishay_IM-2, F.Cu at (19.7, 22.5)
- added L16: 2,2uH, Inductor_THT:L_Axial_L6.6mm_D2.7mm_P10.16mm_Horizontal_Vishay_IM-2, F.Cu at (19.7, 26.7)
- added L8: 0,47uH, SDR_footprints:Resistor_SMD+THTuniversal_0603to2512_RM10_HandSoldering, F.Cu at (9.30, 156.1)
- added L9: 1uH, SDR_footprints:Resistor_SMD+THTuniversal_0603to2512_RM10_HandSoldering, F.Cu at (9.30, 160.3)
- added Q6: MMBT2222A, Package_TO_SOT_SMD:SOT-23, F.Cu at (163.0, 101.5)
- added Q7: MMBT2222A, Package_TO_SOT_SMD:SOT-23, F.Cu at (-4.40, 169.1)
- added Q8: MMBT2222A, Package_TO_SOT_SMD:SOT-23, F.Cu at (10.2, 177.0)
- added R29: 2..4.7k, SDR_footprints:R_1206_0603, F.Cu at (-16.6, 143.5)
- added R30: 10k, SDR_footprints:R_1206_0603, F.Cu at (23.2, 162.7)
- added R31: 2..4.7k, SDR_footprints:R_1206_0603, F.Cu at (-16.6, 138.8)
- added R32: 10k, Resistor_SMD:R_0603_1608Metric_Pad0.98x0.95mm_HandSolder, F.Cu at (3.55, 162.7)
- added R35: 10k, Resistor_SMD:R_0603_1608Metric_Pad0.98x0.95mm_HandSolder, F.Cu at (15.9, 32.4)
- added U7: 74LVC74, Package_SO:TSSOP-14_4.4x5mm_P0.65mm, F.Cu at (37.8, 26.1)
- added Y1: 25Mhz, Crystal:Crystal_HC49-U_Vertical, B.Cu at (53.2, 18.4)
- C23, C24, C25: footprint Capacitor_SMD:C_0603_1608Metric_Pad1.08x0.95mm_HandSolder -> SDR_footprints:C_1206_0603
- L5, L6, L7: footprint Inductor_SMD:L_1210_3225Metric_Pad1.42x2.65mm_HandSolder -> SDR_footprints:Resistor_SMD+THTuniversal_0603to2512_RM10_HandSoldering
- Q1, Q5: value DTC143Z -> MMBT2222A; footprint Package_TO_SOT_SMD:SOT-523 -> Package_TO_SOT_SMD:SOT-23
- R28: footprint Resistor_SMD:R_0603_1608Metric_Pad0.98x0.95mm_HandSolder -> SDR_footprints:R_1206_0603
- moved Q1 225.4 mm to (25.6, 31.2)
- moved Q5 169.7 mm to (15.3, 169.1)
- moved U8 150.9 mm to (51.2, 23.8), turned to -90 degrees
- moved D2 115.7 mm to (174.2, 126.2), turned to -90 degrees
- moved L6 106.8 mm to (167.0, 122.0), turned to 180 degrees
- moved L7 103.1 mm to (176.2, 116.6), turned to -90 degrees
- moved C24 98.5 mm to (168.8, 117.8), turned to 180 degrees
- moved L5 96.6 mm to (167.0, 106.2), turned to 180 degrees
- moved D3 94.5 mm to (176.5, 103.8), turned to 90 degrees
- moved C25 92.0 mm to (172.5, 110.8), turned to -90 degrees
- moved R28 75.3 mm to (159.0, 101.8), turned to -90 degrees
Connections:
- L5 pad 2: Net-(Q5-C) -> Net-(Q6-C)
- L6 pad 2: Net-(Q5-C) -> Net-(Q6-C)
- Q1 pad 1: 74HC4053_RX_TX -> Net-(Q1-B)
- Q5 pad 1: BPF_10_17M -> Net-(Q5-B)
- R28 pad 2: Net-(Q5-C) -> Net-(Q6-C)
- R7 pad 2: Net-(Q1-C) -> Net-(Q8-C)
- U3 pad 10: Net-(Q1-C) -> Net-(Q8-C)
- U3 pad 11: Net-(Q1-C) -> Net-(Q8-C)
- U3 pad 9: Net-(Q1-C) -> Net-(Q8-C)
- U4 pad 10: Net-(Q1-C) -> Net-(Q8-C)
- U4 pad 11: Net-(Q1-C) -> Net-(Q8-C)
- U4 pad 9: Net-(Q1-C) -> Net-(Q8-C)
- U6 pad 28: unconnected-(U6-IO35-Pad28) -> BPF_10_17M
- U6 pad 29: unconnected-(U6-IO36-Pad29) -> BPF_20M
- U6 pad 30: unconnected-(U6-IO37-Pad30) -> BPF_40M
- U6 pad 31: unconnected-(U6-IO38-Pad31) -> BPF_80M
- U8 pad 1: unconnected-(U8-VDD-Pad1) -> +3.3V
- U8 pad 10: unconnected-(U8-CLK0-Pad10) -> Net-(U7A-C)
- U8 pad 2: unconnected-(U8-XA-Pad2) -> Net-(U8-XA)
- U8 pad 3: unconnected-(U8-XB-Pad3) -> Net-(U8-XB)
- U8 pad 4: unconnected-(U8-SCL-Pad4) -> I2C_SCL
- U8 pad 5: unconnected-(U8-SDA-Pad5) -> I2C_SDA
- U8 pad 6: unconnected-(U8-CLK2-Pad6) -> SI5351_CLK2
- U8 pad 7: unconnected-(U8-VDDO-Pad7) -> +3.3VA
- U8 pad 8: unconnected-(U8-GND-Pad8) -> GND
- U8 pad 9: unconnected-(U8-CLK1-Pad9) -> SI5351_CLK1
