File: pure.kicad_pcb (KiCad board)
At the start: 2 copper layers, 100 x 90 mm, 122 parts, among them J1 LINE_IN, J2 USB_B, J3 Program_USB_JTAG, K1 RS-12, Q1 MMBT2222A, Q2 DTC143Z, Q3 BSS138, Q4 BSS138, Q5 MMBT2222A, Q6 MMBT2222A, Q7 MMBT2222A, Q8 MMBT2222A, U1 SN74LVC1G3157DBVR, U11 CH340C, U2 SN74LVC1G3157DBVR, U3 74HC4053, U4 74HC4053, U5 MC33079, U6 ESP32-S3-WROOM-1-N16R8, U7 74LVC74, U8 Si5351A-B-GT, U9 M24C01-WMN, Y1 25Mhz

Commit message: progress in PCB, schematics some footprints are still missing
Parts:
- removed J1: LINE_IN, Connector_Audio:Jack_3.5mm_CUI_SJ1-3525N_Horizontal
- added C55: 390pF, Capacitor_SMD:C_0603_1608Metric_Pad1.08x0.95mm_HandSolder, F.Cu at (252.1, 115.0)
- added C56: 390pF, Capacitor_SMD:C_0603_1608Metric_Pad1.08x0.95mm_HandSolder, F.Cu at (252.1, 117.5)
- added C63: 22..47nF, SDR_footprints:C_1206_0603, F.Cu at (238.3, 127.5)
- added C64: 100nF, SDR_footprints:C_1206_0603, F.Cu at (238.3, 119.8)
- added C65: 10uF, Capacitor_Tantalum_SMD:CP_EIA-3216-18_Kemet-A_Pad1.58x1.35mm_HandSolder, F.Cu at (238.9, 124.7)
- added C66: 100nF, SDR_footprints:C_1206_0603, F.Cu at (238.3, 130.1)
- added C67: 100nF, SDR_footprints:C_1206_0603, F.Cu at (169.5, 132.5)
- added C68: 120pF, Capacitor_SMD:C_0603_1608Metric_Pad1.08x0.95mm_HandSolder, F.Cu at (213.1, 15.0)
- added C69: 22..47nF, SDR_footprints:C_1206_0603, F.Cu at (91.4, 3.98)
- added C71: 100nF, SDR_footprints:C_1206_0603, F.Cu at (185.0, 132.5)
- added C72: 120pF, Capacitor_SMD:C_0603_1608Metric_Pad1.08x0.95mm_HandSolder, F.Cu at (190.0, 142.5)
- added C73: 220pF, SDR_footprints:C_1206_0603, F.Cu at (195.5, 135.8)
- added C75: 3,3nF, SDR_footprints:C_1206_0603, F.Cu at (186.0, 144.0)
- added C76: 3,3nF, SDR_footprints:C_1206_0603, F.Cu at (186.0, 150.0)
- added C77: 10uF, Capacitor_THT:CP_Radial_D5.0mm_P2.00mm, F.Cu at (211.5, 0.68)
- added C78: 100nF, SDR_footprints:C_1206_0603, F.Cu at (213.4, 7.21)
- added C79: 100uF, Capacitor_THT:CP_Radial_D6.3mm_P2.50mm, F.Cu at (192.4, -12.2)
- added C80: 100uF, Capacitor_THT:CP_Radial_D6.3mm_P2.50mm, F.Cu at (192.4, -4.33)
- added C81: 100nF, SDR_footprints:C_1206_0603, F.Cu at (213.4, 9.81)
- added C82: 100uF, Capacitor_THT:CP_Radial_D6.3mm_P2.50mm, F.Cu at (192.4, 3.52)
- added C83: 100nF, SDR_footprints:C_1206_0603, F.Cu at (213.4, 12.4)
- added C84: 100uF, Capacitor_THT:CP_Radial_D6.3mm_P2.50mm, F.Cu at (192.4, 11.4)
- added D10: SS14, Diode_SMD:D_SMA, F.Cu at (81.3, 25.5)
- added D11: LL4148, Diode_SMD:D_MiniMELF, F.Cu at (92.1, 1.01)
- added J10: AudioJack3_Ground_SwitchTR, Connector_Audio:Jack_3.5mm_CUI_SJ1-3525N_Horizontal, B.Cu at (92.8, 41.5)
- added J4: LINE_IN, Connector_Audio:Jack_3.5mm_CUI_SJ1-3525N_Horizontal, B.Cu at (149.0, 42.0)
- added J5: INPUT_OUTPUT, Connector_Coaxial:U.FL_Molex_MCRF_73412-0110_Vertical, B.Cu at (188.0, 153.5)
- added J6: Conn_01x01, MountingHole:MountingHole_3.2mm_M3_DIN965_Pad, B.Cu at (55.0, 154.0)
- added J7: Conn_01x01, MountingHole:MountingHole_3.2mm_M3_DIN965_Pad, B.Cu at (197.0, 154.0)
- added J8: Conn_01x01, MountingHole:MountingHole_3.2mm_M3_DIN965_Pad, B.Cu at (197.0, 42.0)
- added J9: Conn_01x01, MountingHole:MountingHole_3.2mm_M3_DIN965_Pad, B.Cu at (55.0, 42.0)
- added K2: RS-12, Relay_THT:Relay_DPDT_Omron_G5V-2, B.Cu at (181.0, 124.9)
- added L23: 0,22uH, SDR_footprints:Resistor_SMD+THTuniversal_0603to2512_RM10_HandSoldering, F.Cu at (194.0, 132.5)
- added L24: 0,22uH, SDR_footprints:Resistor_SMD+THTuniversal_0603to2512_RM10_HandSoldering, F.Cu at (194.0, 139.0)
- added L25: 4,7uH, SDR_footprints:Resistor_SMD+THTuniversal_0603to2512_RM10_HandSoldering, F.Cu at (194.0, 147.0)
- added L27: 0,22uH, Resistor_THT:R_Axial_DIN0207_L6.3mm_D2.5mm_P10.16mm_Horizontal, F.Cu at (199.2, 7.93)
- added L28: 0,22uH, Resistor_THT:R_Axial_DIN0207_L6.3mm_D2.5mm_P10.16mm_Horizontal, F.Cu at (199.2, 12.0)
- added Q9: MMBT2222A, Package_TO_SOT_SMD:SOT-23, F.Cu at (243.2, 128.6)
- added R40: 1, SDR_footprints:R_1206_0603, F.Cu at (252.4, 104.3)
- added R44: 1, SDR_footprints:R_1206_0603, F.Cu at (252.4, 107.0)
- added R47: 1, SDR_footprints:R_1206_0603, F.Cu at (252.4, 109.7)
- added R48: 1, SDR_footprints:R_1206_0603, F.Cu at (252.4, 112.4)
- added R53: 2..4.7k, SDR_footprints:R_1206_0603, F.Cu at (243.1, 132.2)
- added R54: 2..4.7k, SDR_footprints:R_1206_0603, F.Cu at (91.3, 11.2)
- added R55: 1.0R, SDR_footprints:R_1206_0603, F.Cu at (211.6, -14.8)
- added R56: 1k, SDR_footprints:R_1206_0603, F.Cu at (173.0, 147.2)
- added R57: 1k, SDR_footprints:R_1206_0603, F.Cu at (177.2, 142.5)
- added R58: 1k, SDR_footprints:R_1206_0603, F.Cu at (181.5, 147.2)
- added R59: 1k, SDR_footprints:R_1206_0603, F.Cu at (178.8, 147.2)
- added R60: 1k, SDR_footprints:R_1206_0603, F.Cu at (177.2, 139.8)
- added R61: 1k, SDR_footprints:R_1206_0603, F.Cu at (175.8, 147.2)
- added R62: 18k, SDR_footprints:R_1206_0603, F.Cu at (211.6, -12.1)
- added R63: 11k, SDR_footprints:R_1206_0603, F.Cu at (211.6, -9.35)
- added R64: 150, SDR_footprints:R_1206_0603, F.Cu at (211.6, -6.65)
- added R65: 1K, SDR_footprints:R_1206_0603, F.Cu at (211.6, -3.95)
- added U12: LM317_TO-220, Package_TO_SOT_THT:TO-220-3_Horizontal_TabDown, F.Cu at (200.8, 4.13)
- added U14: MC34063AD, Package_SO:SOIC-8_3.9x4.9mm_P1.27mm, F.Cu at (128.0, 30.3)
- C17: footprint Capacitor_SMD:C_0603_1608Metric_Pad1.08x0.95mm_HandSolder -> SDR_footprints:C_1206_0603
- Q2: value DTC143Z -> MMBT2222A; footprint Package_TO_SOT_SMD:SOT-523 -> Package_TO_SOT_SMD:SOT-23
- R24, R25: footprint Resistor_SMD:R_0603_1608Metric_Pad0.98x0.95mm_HandSolder -> SDR_footprints:R_1206_0603
- moved R29 188.8 mm to (165.8, 94.5), turned to 90 degrees
- moved L9 133.4 mm to (141.5, 142.2), turned to 90 degrees
- moved L10 127.7 mm to (133.2, 133.8), turned to 180 degrees
- moved Q2 124.1 mm to (91.3, 7.68)
- moved L8 123.9 mm to (133.0, 148.2), turned to 180 degrees
- moved U9 113.9 mm to (81.5, 88.2)
- moved R26 113.8 mm to (86.0, 49.5), turned to 180 degrees
- moved C28 113.5 mm to (136.0, 145.0)
- moved C26 111.0 mm to (148.8, 128.5), turned to 180 degrees
- moved C27 110.9 mm to (132.8, 138.0), turned to 180 degrees
- moved R27 103.7 mm to (99.8, 49.5), turned to 180 degrees
- moved J2 77.2 mm to (73.3, 52.7), turned to 90 degrees
- moved D3 51.8 mm to (162.0, 153.5), turned to -90 degrees
- moved L5 45.7 mm to (153.0, 149.8)
- moved C25 38.4 mm to (157.8, 146.2), turned to 0 degrees
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Connections:
- Q2 pad 1: PREAMP -> Net-(Q2-B)
- Q2 pad 3: Net-(D1-A) -> Net-(D11-A)
- U6 pad 10: unconnected-(U6-IO17-Pad10) -> MCU_ATT
- U6 pad 12: KEYBOARD3 -> I2C_SDA
- U6 pad 17: KEYBOARD4 -> I2C_SCL
- U6 pad 18: ENCODER_A -> EEPROM_WP
- U6 pad 20: unconnected-(U6-IO12-Pad20) -> ENCODER_A
- U6 pad 25: EEPROM_WP -> unconnected-(U6-IO48-Pad25)
- U6 pad 34: I2C_SCL -> KEYBOARD4
- U6 pad 35: I2C_SDA -> KEYBOARD3
Routing:
- removed copper zone on B.Cu, net GND
- removed copper zone on F.Cu, net GND
Other:
- board size 100 x 90 mm -> 150 x 120 mm

Commit message: progress on PCB
Parts:
- added C1: 2.2nF, SDR_footprints:C_1206_0603, F.Cu at (164.2, 116.0)
- added C3: 2.2nF, SDR_footprints:C_1206_0603, F.Cu at (164.2, 111.2)
- added C44: 100nF, SDR_footprints:C_1206_0603, F.Cu at (88.3, 143.2)
- added C47: 22..47nF, SDR_footprints:C_1206_0603, F.Cu at (88.2, 130.0)
- added C5: 2.2nF, SDR_footprints:C_1206_0603, F.Cu at (164.2, 102.8)
- added C52: 100nF, SDR_footprints:C_1206_0603, F.Cu at (73.5, 144.8)
- added C53: 100nF, SDR_footprints:C_1206_0603, F.Cu at (73.5, 147.4)
- added C54: 10uF, Capacitor_Tantalum_SMD:CP_EIA-3216-18_Kemet-A_Pad1.58x1.35mm_HandSolder, F.Cu at (68.0, 145.1)
- added C7: 2.2nF, SDR_footprints:C_1206_0603, F.Cu at (164.2, 98.2)
- added L18: 100uH, Inductor_THT:L_Axial_L5.3mm_D2.2mm_P10.16mm_Horizontal_Vishay_IM-1, B.Cu at (66.5, 137.9)
- added L19: 100uH, Inductor_THT:L_Axial_L5.3mm_D2.2mm_P10.16mm_Horizontal_Vishay_IM-1, B.Cu at (66.5, 141.6)
- added R2: 20R, SDR_footprints:R_1206_0603, F.Cu at (168.0, 109.0)
- added R3: 20R, SDR_footprints:R_1206_0603, F.Cu at (168.0, 105.0)
- added R33: 2..4.7k, SDR_footprints:R_1206_0603, F.Cu at (107.5, 127.0)
- added R36: 2..4.7k, SDR_footprints:R_1206_0603, F.Cu at (91.8, 127.5)
- added R37: 1k, Resistor_SMD:R_0603_1608Metric_Pad0.98x0.95mm_HandSolder, F.Cu at (78.1, 144.7)
- added R38: 1k, Resistor_SMD:R_0603_1608Metric_Pad0.98x0.95mm_HandSolder, F.Cu at (78.1, 147.2)
- added R4: 20R, SDR_footprints:R_1206_0603, F.Cu at (168.0, 100.5)
- added U10: MC33079, Package_SO:SOIC-14_3.9x8.7mm_P1.27mm, F.Cu at (124.8, 86.9)
- C34: footprint SDR_footprints:C_1206_0603 -> Capacitor_SMD:C_0603_1608Metric_Pad1.08x0.95mm_HandSolder
- C77, C79, C80, C82, C84, L27, L28, U12: moved to B.Cu
- L1, L2: footprint Inductor_SMD:L_1210_3225Metric_Pad1.42x2.65mm_HandSolder -> Inductor_THT:L_Axial_L5.3mm_D2.2mm_P10.16mm_Horizontal_Vishay_IM-1
- L14, L15, L16: footprint Inductor_THT:L_Axial_L6.6mm_D2.7mm_P10.16mm_Horizontal_Vishay_IM-2 -> SDR_footprints:Resistor_SMD+THTuniversal_0603to2512_RM10_HandSoldering
- R1: footprint Resistor_SMD:R_0603_1608Metric_Pad0.98x0.95mm_HandSolder -> SDR_footprints:R_1206_0603
- R28, R30: footprint SDR_footprints:R_1206_0603 -> Resistor_SMD:R_0603_1608Metric_Pad0.98x0.95mm_HandSolder
- moved Q8 188.0 mm to (144.5, 89.5)
- moved C50 172.7 mm to (197.8, 98.0), turned to -90 degrees
- moved C49 169.9 mm to (192.0, 105.2), turned to 90 degrees
- moved U7 167.1 mm to (182.5, 106.2)
- moved R31 165.0 mm to (129.5, 126.8), turned to 90 degrees
- moved U8 162.3 mm to (192.5, 99.0)
- moved Y1 161.7 mm to (194.8, 90.9)
- moved C51 160.4 mm to (185.2, 99.8), turned to 90 degrees
- moved D5 159.7 mm to (142.5, 134.8), turned to 90 degrees
- moved D7 156.0 mm to (118.8, 134.8), turned to 90 degrees
- moved D4 154.0 mm to (144.5, 154.2)
- moved C21 154.0 mm to (61.5, 44.2), turned to -90 degrees
- moved L12 153.9 mm to (123.5, 145.8), turned to 90 degrees
- moved D6 153.4 mm to (124.2, 154.2)
- moved C37 147.7 mm to (106.2, 135.0), turned to -90 degrees
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Connections:
- R11 pad 1: Net-(K1-Pad8) -> Net-(U5C--)
- R11 pad 2: Net-(U5C--) -> Net-(K1-Pad8)

Commit message: progress on schematics and pcb
Parts:
- added R39: 4,7k, Resistor_SMD:R_0603_1608Metric_Pad0.98x0.95mm_HandSolder, F.Cu at (120.0, 83.0)
- added R41: 4,7k, Resistor_SMD:R_0603_1608Metric_Pad0.98x0.95mm_HandSolder, F.Cu at (112.5, 86.0)
- added R42: 4,7k, Resistor_SMD:R_0603_1608Metric_Pad0.98x0.95mm_HandSolder, F.Cu at (108.0, 83.0)
- added R43: 4,7k, Resistor_SMD:R_0603_1608Metric_Pad0.98x0.95mm_HandSolder, F.Cu at (108.0, 75.0)
- added R45: 4,7k, Resistor_SMD:R_0603_1608Metric_Pad0.98x0.95mm_HandSolder, F.Cu at (112.5, 72.0)
- added R46: 4,7k, Resistor_SMD:R_0603_1608Metric_Pad0.98x0.95mm_HandSolder, F.Cu at (120.0, 75.0)
- added R49: 1k, Resistor_SMD:R_0603_1608Metric_Pad0.98x0.95mm_HandSolder, F.Cu at (216.6, 88.0)
- added R50: 1k, Resistor_SMD:R_0603_1608Metric_Pad0.98x0.95mm_HandSolder, F.Cu at (216.6, 90.5)
- L1, L2: moved to B.Cu
- moved C56 153.2 mm to (105.0, 75.0), turned to -90 degrees
- moved C55 150.6 mm to (105.0, 83.0), turned to 90 degrees
- moved C10 136.6 mm to (172.8, 97.5)
- moved C11 133.4 mm to (187.2, 118.4), turned to 90 degrees
- moved C12 129.3 mm to (190.8, 118.2), turned to -90 degrees
- moved C9 128.2 mm to (172.8, 106.1), turned to 90 degrees
- moved L1 127.3 mm to (179.0, 88.7), turned to -90 degrees
- moved R6 122.7 mm to (188.8, 113.8)
- moved R5 122.5 mm to (187.8, 110.3), turned to -90 degrees
- moved R44 118.5 mm to (134.0, 112.5), turned to 180 degrees
- moved R40 117.4 mm to (135.0, 105.0), turned to 180 degrees
- moved L2 116.3 mm to (184.8, 116.2), turned to 180 degrees
- moved C15 98.4 mm to (155.0, 86.8), turned to -90 degrees
- moved C14 81.2 mm to (155.0, 104.8), turned to -90 degrees
- moved C18 66.0 mm to (132.3, 62.6), turned to 90 degrees
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Routing:
- net RX180: track 0.00 -> 36.1 mm
- net RX90: track 0.00 -> 31.8 mm, vias 0 -> 2
- net Net-(C13-Pad2): track 0.00 -> 29.0 mm, vias 0 -> 2
- net Net-(U5A--): track 0.00 -> 24.1 mm
- net Net-(U5D--): track 0.00 -> 23.6 mm
- net Net-(U5B--): track 0.00 -> 19.2 mm
- net P270: track 0.00 -> 18.0 mm
- net Net-(U5C--): track 0.00 -> 17.0 mm
- net Net-(U1B-V+): track 0.00 -> 15.7 mm
- net P90: track 0.00 -> 15.3 mm, vias 0 -> 2
- net Net-(R19-Pad2): track 0.00 -> 6.51 mm
- net J90: track 0.00 -> 6.28 mm
- net RX270: track 0.00 -> 6.27 mm
- net Net-(R12-Pad1): track 0.00 -> 6.08 mm
- net RX0: track 0.00 -> 5.77 mm
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