File: PA.kicad_sch (KiCad schematic)
At the start: 29 parts, among them J7 ANT, K1 TQ2-12VDC, K2 RS-12, Q3 MMBT2222, Q4 BD139, T1 Transformer_1P_1S

Commit message: finich IF_RX_Schematics, begin MCU, delete *.sch files
Parts:
- removed C37: 15nF, LCSDR:C_0603_HandSoldering, symbol C_Small
- removed C38: 47nF, LCSDR:C_1206_0603, symbol C_Small
- removed C39: 100nF, LCSDR:C_1206, symbol C_Small
- removed C41, C43: 100nF, LCSDR:C_1206_0603, symbol C_Small
- removed C48, C49: 100nF, LCSDR:C_Disc_D7.5mm_W2.5mm_P5.00mm, symbol C_Small
- removed C52, C55: 1nF, LCSDR:C_Disc_D7.5mm_W2.5mm_P5.00mm, symbol C_Small
- removed C?: 47pF, LCSDR:C_Disc_D7.5mm_W2.5mm_P5.00mm, symbol C_Small
- removed D1: LL4148, Diodes_SMD:D_MiniMELF, symbol D_Small
- removed E1: SPARK_GAP, LCSDR:C_Rect_L11.0mm_W8.8mm_P10.00mm_MKT, symbol SPARK_GAP
- removed J7: ANT, Connectors:SMA_THT_Jack_Straight, symbol Conn_Coaxial
- removed K1: TQ2-12VDC, Relays_THT:Relay_DPDT_FRT5, symbol TQ2-12VDC
- removed K2: RS-12, Relays_THT:Relay_DPDT_FRT5, symbol RS-12
- removed L14, L?: 1uH, Inductors_THT:L_Axial_L12.8mm_D5.8mm_P20.32mm_Horizontal_Fastron_HBCC, symbol L_Small
- removed Q3: MMBT2222, LCSDR:SOT-23, symbol Q_NPN_BEC
- removed Q4: BD139, TO_SOT_Packages_THT:TO-126_Vertical, symbol BD139
- removed Q?: 2SC5706, TO_SOT_Packages_SMD:TO-252-2, symbol Q_NPN_BCE
- removed R10: 10, LCSDR:R_1206_0603, symbol R_Small
- removed R11: 2.2k, LCSDR:R_1206_0603, symbol R_Small
- removed R16: 470, LCSDR:R_1206_0603, symbol R_Small
- removed R20: 56, LCSDR:R_0603_HandSoldering, symbol R_Small
- removed R21: 1k, LCSDR:R_0603_HandSoldering, symbol R_Small
- removed R22, R23: 10k, LCSDR:R_1206_0603, symbol R_Small
- removed R39: 5.1, LCSDR:R_0603_HandSoldering, symbol R_Small
- removed T1: Transformer_1P_1S, symbol Transformer_1P_1S
