File: PowerSupply.kicad_sch (KiCad schematic)
At the start: 7 parts, among them J8 Jack-DC, U5 AP1117-33, U6 AP1117-50

Commit message: progress in PCB, schematics some footprints are still missing
Parts:
- removed C24, C57: 220uF, LCSDR:C_Radial_D5_L11_P2.5, symbol CP_Small
- removed C60, C61: 100uF, Capacitors_THT:CP_Radial_D6.3mm_P2.50mm, symbol CP_Small
- removed J8: Jack-DC, LCSDR:BARREL_JACK, symbol Jack-DC
- removed U5: AP1117-33, TO_SOT_Packages_SMD:SOT-223-3Lead_TabPin2, symbol AP1117-33
- removed U6: AP1117-50, TO_SOT_Packages_SMD:SOT-223-3Lead_TabPin2, symbol AP1117-50
- added C68: 120pF, Capacitor_SMD:C_0603_1608Metric_Pad1.08x0.95mm_HandSolder, symbol Device:C_Small
- added C70: 1000uF, symbol Device:C_Polarized_Small
- added C77: 10uF, Capacitor_THT:CP_Radial_D5.0mm_P2.00mm, symbol Device:C_Polarized_Small
- added C78, C81, C83: 100nF, SDR_footprints:C_1206_0603, symbol Device:C_Small
- added C79, C80, C82, C84: 100uF, Capacitor_THT:CP_Radial_D6.3mm_P2.50mm, symbol Device:C_Polarized_Small
- added D10: SS14, Diode_SMD:D_SMA, symbol Diode:SS14
- added L26: 100uH, symbol Device:L_Small
- added L27, L28: 0,22uH, Resistor_THT:R_Axial_DIN0207_L6.3mm_D2.5mm_P10.16mm_Horizontal, symbol Device:L_Small
- added R55: 1.0R, SDR_footprints:R_1206_0603, symbol Device:R_Small
- added R62: 18k, SDR_footprints:R_1206_0603, symbol Device:R_Small
- added R63: 11k, SDR_footprints:R_1206_0603, symbol Device:R_Small
- added R64: 150, SDR_footprints:R_1206_0603, symbol Device:R_Small
- added R65: 1K, SDR_footprints:R_1206_0603, symbol Device:R_Small
- added U12: LM317_TO-220, Package_TO_SOT_THT:TO-220-3_Horizontal_TabDown, symbol Regulator_Linear:LM317_TO-220
- added U14: MC34063AD, Package_SO:SOIC-8_3.9x4.9mm_P1.27mm, symbol Regulator_Switching:MC34063AD
Connections:
- new net: D10.1 (K), L26.1, U14.2 (SwE)
- new net: C70.1, C78.1, L26.2, L27.1, L28.1, R62.1
- new net: R62.2, R63.1, U14.5 (Vfb)
- new net: C81.1, C82.1, R64.2, R65.1, U12.1 (ADJ)
- new net: C68.2, U14.3 (TC)
- new net: R55.2, U14.1 (SwC), U14.7 (Ipk), U14.8 (DC)
- new net +10V: C84.1, R64.1, U12.2 (VO)
- new net +12V: C77.1, C83.1, R55.1, U12.3 (VI), U14.6 (Vin)
- new net +3.3V: C79.1, L28.2
- new net +3.3VA: C80.1, L27.2
- new net GND: C68.1, C70.2, C77.2, C78.2, C79.2, C80.2, C81.2, C82.2, C83.2, C84.2, D10.2 (A), R63.2, R65.2, U14.4 (GND)
