File: 20M.kicad_sch (KiCad schematic)
At the start: 13 parts, among them Q5 MMBT2222A

Commit message: progress on PCB
Parts:
- R30: footprint SDR_footprints:R_1206_0603 -> Resistor_SMD:R_0603_1608Metric_Pad0.98x0.95mm_HandSolder
Changed lines of the file:
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@@
 			)
 		)
-		(property "Footprint" "SDR_footprints:R_1206_0603"
+		(property "Footprint" "Resistor_SMD:R_0603_1608Metric_Pad0.98x0.95mm_HandSolder"
 			(at 88.9 104.14 0)
 			(effects
