File: IF2.kicad_sch (KiCad schematic)
At the start: 38 parts, among them J5 JACK_TRS_3pins, U3 MC33079

Commit message: add custom footprints, progress on schema and PCB
Parts:
- removed C10, C13, C21, C34, C40, C7: 10uF, LCSDR:CP_Radial_D5.0mm_P2.00mm, symbol CP_Small
- removed C11, C12, C29, C30, C87, C88: 27nF, Capacitors_SMD:C_0603_HandSoldering, symbol C_Small
- removed C23, C26: 100nF, Capacitors_SMD:C_0603_HandSoldering, symbol C_Small
- removed C71, C72: 2.2uF, LCSDR:CP_Radial_D5.0mm_P2.00mm, symbol CP_Small
- removed J5: JACK_TRS_3pins, LCSDR:audio_jack_3_5mm_PJ307, symbol JACK_TRS_3pins
- removed L6, L7: 100uH, Resistors_THT:R_Axial_DIN0204_L3.6mm_D1.6mm_P7.62mm_Horizontal, symbol L_Small
- removed L8, L9: 4.7mH, LCSDR:R_Axial_DIN0207_L6.3mm_D2.5mm_P10.16mm_Horizontal, symbol L_Small
- removed R1, R26, R29, R31, R4, R65: 10k, LCSDR:R_0603_HandSoldering, symbol R_Small
- removed R12, R19: 33, LCSDR:R_0603_HandSoldering, symbol R_Small
- removed R13, R28: 330, Resistors_SMD:R_0603_HandSoldering, symbol R_Small
- removed R18, R27: 330, LCSDR:R_0603_HandSoldering, symbol R_Small
- removed R25, R9: 33, Resistors_SMD:R_0603_HandSoldering, symbol R_Small
- removed R67, R69: 1k, LCSDR:R_1206_0603, symbol R_Small
- removed U3: MC33079, Housings_SOIC:SOIC-14_3.9x8.7mm_Pitch1.27mm, symbol MC33079

Commit message: progress in PCB, schematics some footprints are still missing
Parts:
- added C55, C56: 390pF, Capacitor_SMD:C_0603_1608Metric_Pad1.08x0.95mm_HandSolder, symbol Device:C_Small
- added C57: 100nF, symbol Device:C_Small
- added C58: 10uF, symbol Device:C_Polarized_Small
- added C59, C62: 4,7uF, symbol Device:C_Polarized_Small
- added C60, C61: 10nF, symbol Device:C_Small
- added C64: 100nF, SDR_footprints:C_1206_0603, symbol Device:C_Small
- added J4: LINE_IN, Connector_Audio:Jack_3.5mm_CUI_SJ1-3525N_Horizontal, symbol Connector_Audio:AudioJack2_Ground_Switch
- added L20: 100uH, symbol Device:L_Small
- added L21, L22: 4.7mH, symbol Device:L_Small
- added R39, R41, R42, R43, R45, R46: 4,7k, symbol Device:R_Small
- added R40, R44, R47, R48: 1, SDR_footprints:R_1206_0603, symbol Device:R_Small
- added R49, R50: 1k, symbol Device:R_Small
- added R51, R52: 10k, symbol Device:R_Small
- added U10: MC33079, symbol Amplifier_Operational:MC33079
Connections:
- new net: R39.1, R40.2, U10.8
- new net: R39.2, R41.2, U10.9 (-)
- new net: C56.1, R43.1, R45.1, R48.2, U10.1
- new net: C61.2, C62.2, L22.1
- new net: C55.1, R41.1, R42.1, R44.2, U10.7
- new net: C59.1, R50.2
- new net: C59.2, C60.2, L21.1
- new net: C57.1, C58.1, L20.2, U10.4 (V+)
- new net: C56.2, R43.2, R49.1, U10.2 (-)
- new net: R45.2, R46.2, U10.13 (-)
- new net: C55.2, R42.2, R50.1, U10.6 (-)
- new net: R46.1, R47.2, U10.14
- new net: C62.1, R49.2
- new net +10V: L20.1
- new net +5V: C64.2, U10.10 (+), U10.12 (+), U10.3 (+), U10.5 (+)
- new net GND: C57.2, C58.2, C60.1, C61.1, C64.1, J4.G, R51.1, R52.1, U10.11 (V-)
- new net TX0: R44.1
- new net TX180: R40.1
- new net TX270: R47.1
- new net TX90: R48.1
- new net TX_IQ_I: J4.S, J4.SN, L22.2, R52.2
- new net TX_IQ_Q: J4.T, J4.TN, L21.2, R51.2

Commit message: progress on PCB
Parts:
- U10: footprint (none) -> Package_SO:SOIC-14_3.9x8.7mm_P1.27mm
Changed lines of the file:
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@@
 			)
 		)
-		(property "Footprint" ""
+		(property "Footprint" "Package_SO:SOIC-14_3.9x8.7mm_P1.27mm"
 			(at 114.3 35.56 0)
 			(effects
@@
 			)
 		)
-		(property "Footprint" ""
+		(property "Footprint" "Package_SO:SOIC-14_3.9x8.7mm_P1.27mm"
 			(at 62.23 143.51 0)
 			(effects
@@
 			)
 		)
-		(property "Footprint" ""
+		(property "Footprint" "Package_SO:SOIC-14_3.9x8.7mm_P1.27mm"
 			(at 193.04 78.74 0)
 			(effects
@@
 			)
 		)
-		(property "Footprint" ""
+		(property "Footprint" "Package_SO:SOIC-14_3.9x8.7mm_P1.27mm"
 			(at 114.3 73.66 0)
 			(effects
@@
 			)
 		)
-		(property "Footprint" ""
+		(property "Footprint" "Package_SO:SOIC-14_3.9x8.7mm_P1.27mm"
 			(at 193.04 44.45 0)
 			(effects

Commit message: progress on schematics and pcb
Parts:
- R39, R41, R42, R43, R45, R46, R49, R50: footprint (none) -> Resistor_SMD:R_0603_1608Metric_Pad0.98x0.95mm_HandSolder
Changed lines of the file:
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@@
 			)
 		)
-		(property "Footprint" ""
+		(property "Footprint" "Resistor_SMD:R_0603_1608Metric_Pad0.98x0.95mm_HandSolder"
 			(at 111.76 60.96 0)
 			(effects
@@
 			)
 		)
-		(property "Footprint" ""
+		(property "Footprint" "Resistor_SMD:R_0603_1608Metric_Pad0.98x0.95mm_HandSolder"
 			(at 190.5 33.02 0)
 			(effects
@@
 			)
 		)
-		(property "Footprint" ""
+		(property "Footprint" "Resistor_SMD:R_0603_1608Metric_Pad0.98x0.95mm_HandSolder"
 			(at 185.42 58.42 0)
 			(effects
@@
 			)
 		)
-		(property "Footprint" ""
+		(property "Footprint" "Resistor_SMD:R_0603_1608Metric_Pad0.98x0.95mm_HandSolder"
 			(at 130.81 99.06 0)
 			(effects
@@
 			)
 		)
-		(property "Footprint" ""
+		(property "Footprint" "Resistor_SMD:R_0603_1608Metric_Pad0.98x0.95mm_HandSolder"
 			(at 111.76 88.9 0)
 			(effects
@@
 			)
 		)
-		(property "Footprint" ""
+		(property "Footprint" "Resistor_SMD:R_0603_1608Metric_Pad0.98x0.95mm_HandSolder"
 			(at 210.82 39.37 0)
 			(effects
@@
 			)
 		)
-		(property "Footprint" ""
+		(property "Footprint" "Resistor_SMD:R_0603_1608Metric_Pad0.98x0.95mm_HandSolder"
 			(at 189.23 67.31 0)
 			(effects
@@
 			)
 		)
-		(property "Footprint" ""
+		(property "Footprint" "Resistor_SMD:R_0603_1608Metric_Pad0.98x0.95mm_HandSolder"
 			(at 111.76 50.8 0)
 			(effects
